File: PCB/PCB.sch (KiCad schematic (older format))
At the start: 20 parts, among them J1 Conn_01x04_Female, J2 Conn_01x05_Female, J3 Screw_Terminal_01x02, J4 Conn_01x03_Female, J5 Conn_01x03_Female, J6 Conn_01x03_Female, J7 Conn_01x03_Female, U1 R-785.0-1.0

Commit message: Add files via upload
MàJ
Connections:
- net +5V: now also A1.27 (+5V); no longer A1.30 (VIN)
Changed lines of the file:
@@
 L power:+5V #PWR0116
 U 1 1 5F157965
-P 3850 2300
-F 0 "#PWR0116" H 3850 2150 50  0001 C CNN
-F 1 "+5V" H 3865 2473 50  0000 C CNN
-F 2 "" H 3850 2300 50  0001 C CNN
-F 3 "" H 3850 2300 50  0001 C CNN
-	1    3850 2300
+P 4150 2300
+F 0 "#PWR0116" H 4150 2150 50  0001 C CNN
+F 1 "+5V" H 4165 2473 50  0000 C CNN
+F 2 "" H 4150 2300 50  0001 C CNN
+F 3 "" H 4150 2300 50  0001 C CNN
+	1    4150 2300
 	1    0    0    -1
 $EndComp
@@
 NoConn ~ 3450 4000
 NoConn ~ 4050 2300
-NoConn ~ 4150 2300
 $Comp
 L Device:LED D1
@@
 	1    0    0    -1
 $EndComp
+NoConn ~ 3850 2300
 $EndSCHEMATC
